File: Hardware/Basic/Bottom/KickJr-Basic-BOTTOM.sch (EAGLE design)
At the start: 38 parts, among them U3 PCF8523, Y2 32.7680kHz

Commit message: update
Other:
- note added: "Kick Jr PPG Circuit"
- note removed: "Maggie PPG Circuit"
Changed lines of the file:
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@@
 <text x="38.1" y="83.82" size="2.54" layer="97" font="vector" ratio="15">Vref Generator and
 Bypass Capacitors</text>
-<text x="99.06" y="185.42" size="7.62" layer="97" font="vector" ratio="15">Maggie PPG Circuit</text>
+<text x="99.06" y="185.42" size="7.62" layer="97" font="vector" ratio="15">Kick Jr PPG Circuit</text>
 <text x="190.5" y="15.24" size="4.572" layer="97" font="vector" ratio="15">Real-Time Clock (RTC)</text>
 <text x="226.06" y="-12.7" size="1.27" layer="97">I2C Address = 0x68h</text>
