File: Hardware/Basic/Top/Maggie-BASIC-TOP.sch (EAGLE design)
At the start: 64 parts, among them SW1 SWITCH.MOM, SW2 SWITCH.MOM, U2 NRF52832_MODULE_MDBT42, U4 FT231XS, U5 PCF8523

Commit message: update
Parts:
- removed C10, C11: 300p, LinnesLab-Passives:CAPACITOR0603
- removed C29: 1u, LinnesLab-Passives:CAPACITOR0603
- removed R17: 100k, LinnesLab-Passives:RESISTOR0603
- removed U5: PCF8523, LinnesLab-Clocks:PCF8523
- removed XTAL3: 32.7680kHz, LinnesLab-Clocks:CRYSTALECS-.327-12.5-12-C-TR
- added J1: (no value), LinnesLab-Connectors:CONN_061.27MM
Connections:
- removed net BATT: R15.1, R16.2
- removed net CD1: SD2.CARD_DETECT
- removed net CHRG.STAT: CHRG2.STAT, R14.1
- removed net CS.OLED: U3./CS
- removed net DC.OLED: U3.DC/I2C_SA0
- removed net N$21: U5.OSCI, XTAL3.2
- removed net RESET.OLED: U3./RES
- removed net SD.CS: SD2.CS
- removed net SW1: SW1.1, SW2.1
- new net A4/BATT: R15.1, R16.2, U2.P0.28/AIN4
- new net A6/TIA: U2.P0.30/AIN6
- new net A7/PPG: U2.P0.31/AIN7
- new net D11/SW1: U2.P0.11
- new net D11/SW2: SW1.1
- new net D15/SW2: SW2.1, U2.P0.15
- new net D16/CS/OLED: U2.P0.16, U3./CS
- new net D27/CHRG.STATUS: CHRG2.STAT, R14.1, U2.P0.27
- new net D29/LED.CTRL: U2.P0.29/AIN5
- new net D3/RESETOLED: U2.P0.03/AIN1, U3./RES
- new net D4/DCOLED: U2.P0.04/AIN2, U3.DC/I2C_SA0
- new net D5/CD1: SD2.CARD_DETECT, U2.P0.05/AIN3
- new net D7/SD.CS: SD2.CS, U2.P0.07
- net 3.3V: now also R8.2, R9.2; no longer C29.1, R17.2, U5.VDD
- net GND: no longer C10.2, C11.2, C29.2, R17.1, U5.VSS
- net N$20: now also U2.P0.02/AIN0; no longer U5.OSCO, XTAL3.1
- net P0.09/NFC1: no longer C11.1
- net P0.10/NFC2: no longer C10.1
- net SCL: now also R8.1; no longer U5.SCL
- net SDA: now also R9.1; no longer U5.SDA
Other:
- note added: "FTDI SERIAL-TO-USB CONVERTER"
- note removed: "___Pins we need___ DIGITAL OUTPUTS CS.OLED RESET.OLED DC.OLED (SPI) (I2C) SP.CS (optional) Card Detect 1 and 2 Digital INPUTS 3X buttons Charge Status ANALOG INPUTS Battery Monitor ANALOG OUTPUTS Data to send to bottom board 3.3V \ GND I2C TIA 2-3x GPIO PPG (Pulse Sensor Circuit Output)"
- moved on the sheet: C12, C4, C5, C6, C7, C8, C9, JP2, L2, LED3, LED4, LED5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

Commit message: update
Parts:
- removed C24, C25: 1u, LinnesLab-Passives:CAPACITOR0603
- removed C26, C27: 4.7u, LinnesLab-Passives:CAPACITOR0603
- removed J1: (no value), LinnesLab-Connectors:CONN_061.27MM
- removed R13: (no value), LinnesLab-Passives:RESISTOR0603
- removed R14: 100k, LinnesLab-Passives:RESISTOR0603
- added C11, C20: 1u, LinnesLab-Passives:CAPACITOR0603
- added C21, C22: 4.7u, LinnesLab-Passives:CAPACITOR0603
- added J3: (no value), LinnesLab-Connectors:CONN_07-1.27MM
- added R21: 5K, LinnesLab-Passives:RESISTOR0603
- added R22: 100k, LinnesLab-Passives:RESISTOR0603
- C18: value 2.2uF -> (none); device LinnesLab-Passives:CAPACITOR0402 -> LinnesLab-Passives:CAPACITOR0603
Connections:
- net !CTS renamed CTS
- removed net !DTR: U4.!DTR
- removed net A4/BATT: R15.1, R16.2, U2.P0.28/AIN4
- removed net A6/TIA: U2.P0.30/AIN6
- removed net A7/PPG: U2.P0.31/AIN7
- removed net D11/SW2: SW1.1
- removed net D27/CHRG.STATUS: CHRG2.STAT, R14.1, U2.P0.27
- removed net D29/LED.CTRL: U2.P0.29/AIN5
- new net 3.3: C12.2, C17.2, C19.2, C4.2, CORTEX1.VCC, D1.C, LED5.A, LED6.A, R5.2, R8.2, R9.2, SD2.VDD, U2.VDD, U3.VBAT, U3.VDD, U4.!RESET, U4.VCCIO
- new net A4/PPG: J3.7, U2.P0.28/AIN4
- new net A5/TIA: J3.6, U2.P0.29/AIN5
- new net A7/BATT: R15.1, R16.2, U2.P0.31/AIN7
- new net CHRG.STAT: CHRG2.STAT, R22.1, U2.P0.27
- new net D30/LED.CTRL: J3.5, U2.P0.30/AIN6
- net 3.3V: now also C20.1, J3.4; no longer C12.2, C17.2, C19.2, C25.1, C4.2, CORTEX1.VCC, D1.C, LED5.A, LED6.A, R5.2, R8.2, R9.2, SD2.VDD, U2.VDD, U3.VBAT, U3.VDD, U4.!RESET, U4.VCCIO
- net D11/SW1: now also SW1.1
- net DTR: now also U4.!DTR
- net GND: now also C11.1, C20.2, C21.2, C22.1, J3.3, R21.1; no longer C24.1, C25.2, C26.2, C27.1, R13.1
- net N$17: now also R21.2; no longer R13.2
- net SCL: now also J3.2
- net SDA: now also J3.1
- net VIN: now also C11.2, C22.2, R22.2; no longer C24.2, C27.2, R14.2
- net VLIPO: now also C21.1; no longer C26.1
Other:
- note added: "HEADERS CONN TOP/BTM BRDS"
- note removed: "REAL-TIME CLOCK"
- moved on the sheet: C12, C7, C8, C9, CHRG2, D4, D5, J2, L2, LDO2, LED3, LED4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
