File: Hardware/Basic/Top/Maggie-BASIC-TOP.brd (EAGLE design)
At the start: 0 parts

Commit message: commit
Parts:
- added C10, C11: 300p, LinnesLab-Passives:C0603
- added C12: 10u, LinnesLab-Passives:C0805
- added C13, C15, C17, C18, C19: 2.2uF, LinnesLab-Passives:C0402
- added C14, C4: 100n, LinnesLab-Passives:C0603
- added C16: 10uF, LinnesLab-Passives:C0603
- added C24, C25, C29, C7: 1u, LinnesLab-Passives:C0603
- added C26, C27: 4.7u, LinnesLab-Passives:C0603
- added C5, C6: 47p, LinnesLab-Passives:C0603
- added C8, C9: (no value), LinnesLab-Passives:C0603
- added CHRG2: MCP73831, LinnesLab-Power:SOT23-5
- added CORTEX1: CORTEX_DEBUG_PTH, LinnesLab-Connectors:2X5-PTH-1.27MM
- added D1, D4, D5: (no value), LinnesLab-DiscreteSemi:USC
- added J2: (no value), LinnesLab-Connectors:1X02
- added JP2: (no value), LinnesLab-Switches:SMT-JUMPER_2_NO_SILK
- added L2: 10u, LinnesLab-Passives:L0603
- added LDO2: MIC5504, LinnesLab-Power:SOT23-5
- added LED3, LED5: RED, LinnesLab-LED:LED-0603
- added LED4: BLUE, LinnesLab-LED:LED-0603
- added LED6: YELLOW, LinnesLab-LED:LED-0603
- added R1, R13, R2: (no value), LinnesLab-Passives:R0603
- added R10, R11: 27, LinnesLab-Passives:R0603
- added R12, R18, R3, R4: 1k, LinnesLab-Passives:R0603
- added R14, R15, R16, R17: 100k, LinnesLab-Passives:R0603
- added R5, R6: 10k, LinnesLab-Passives:R0603
- added R7: 390k, LinnesLab-Passives:R0603
- added R8, R9: 10K, LinnesLab-Passives:R0603
- added SD2: (no value), LinnesLab-Connectors:MICROSD
- added SW1, SW2: SWITCH.MOM, LinnesLab-Switches:TACTILE_SWITCH_SMD_6.2MM_TALL
- added SW3, SW4: (no value), LinnesLab-Switches:BUTTON-GULLWING
- added U2: NRF52832_MODULE_MDBT42, LinnesLab-Microcontrollers:BLE_MODULE_RAYTAC_MDBT42
- added U3: (no value), LinnesLab-Displays:UG-2864HSWEG01_0.96IN_NO-WRAPAROUND
- added U4: FT231XS, LinnesLab-DigitalIC:SSOP20_L
- added U5: PCF8523, LinnesLab-Clocks:SO8
- added USB2: USB.MICRO-BIGGERPADS, LinnesLab-Connectors:USB-MICRO-01.BIGGERPADS
- added XTAL2: 32.768kHz, LinnesLab-Clocks:2-SMD.NOLEAD.2.0MMTO1.2MM
- added XTAL3: 32.7680kHz, LinnesLab-Clocks:2-SMD.NOLEAD.2.0MMTO1.2MM
Connections:
- new net !CTS: JP2.2, U4.9
- new net !DTR: U4.1
- new net 3.3V: C12.2, C17.2, C19.2, C25.1, C29.1, C4.2, CORTEX1.1, D1.-, LDO2.5, LED5.A, LED6.A, R17.2, R5.2, SD2.4, U2.11, U3.6, U3.9, U4.14, U4.3, U5.8
- new net BATT: R15.1, R16.2
- new net CD1: SD2.CD1
- new net CD2: SD2.CD2
- new net CHRG.STAT: CHRG2.1, R14.1
- new net CS.OLED: U3.13
- new net DC.OLED: U3.15
- new net DFU: SW3.3, U2.34
- new net DTR: C14.1
- new net FRST: U2.38
- new net FT3V3: U4.13
- new net GND: C10.2, C11.2, C12.1, C16.1, C17.1, C18.1, C19.1, C24.1, C25.2, C26.2, C27.1, C29.2, C4.1, C5.2, C6.1, C7.2, C8.1, C9.2, CHRG2.2, CORTEX1.3, CORTEX1.5, CORTEX1.7, CORTEX1.9, J2.1, JP2.1, LDO2.2, LED3.C, LED4.C, R13.1, R16.1, R17.1, R6.1, R7.2, SD2.6, SD2.MT1, SD2.MT2, SW1.B1, SW1.B2, SW2.B1, SW2.B2, SW3.1, SW4.3, U2.1, U2.12, U2.24, U2.39, U3.1, U3.10, U3.12, U3.29, U3.30, U3.8, U4.16, U4.6, U5.4, USB2.5, USB2.S1, USB2.S2, USB2.S3, USB2.S4, USB2.S5, USB2.S6
- new net LED1: R3.2, U2.31
- new net LED2: R4.2, U2.33
- new net MISO: SD2.7, U2.28
- new net MOSI: SD2.3, U2.27, U3.19
- new net N$1: R6.2, U3.11
- new net N$10: LED4.A, R4.1
- new net N$11: L2.1, U2.10
- new net N$12: C7.1, L2.2, U2.9
- new net N$13: C16.2, U3.28
- new net N$14: CORTEX1.8
- new net N$15: C18.2, U3.27
- new net N$17: CHRG2.5, R13.2
- new net N$2: R7.1, U3.26
- new net N$20: U5.2, XTAL3.P$1
- new net N$21: U5.1, XTAL3.P$2
- new net N$23: R10.2, U4.12
- new net N$24: R11.2, U4.11
- new net N$25: LED5.C, R12.2
- new net N$26: LED6.C, R18.2
- new net N$3: C13.2, U3.2
- new net N$4: C8.2, U2.13, XTAL2.P$1
- new net N$5: C13.1, U3.3
- new net N$6: C9.1, U2.14, XTAL2.P$2
- new net N$7: C15.2, U3.4
- new net N$8: C15.1, U3.5
- new net N$9: LED3.A, R3.1
- new net P0.09/NFC1: C11.1, U2.22
- new net P0.10/NFC2: C10.1, U2.23
- new net RESET: C14.2, CORTEX1.10, D1.+, R5.1, SW4.1, U2.35
- new net RESET.OLED: U3.14
- new net RXD.FT: R2.1, U4.4
- new net RXD.NRF: R1.2, U2.21
- new net RXLED: R12.1, U4.17
- new net SCK: SD2.5, U2.26, U3.18
- new net SCL: U2.3, U5.6
- new net SD.CS: SD2.2
- new net SDA: U2.2, U5.5
- new net SW1: SW1.A1, SW2.A1
- new net SWCLK: CORTEX1.4, U2.36
- new net SWDIO: CORTEX1.2, U2.37
- new net SWO: CORTEX1.6, U2.32
- new net TXD.FT: R1.1, U4.20
- new net TXD.NRF: R2.2, U2.19
- new net TXLED: R18.1, U4.10
- new net USB+: C5.1, R11.1, USB2.3
- new net USB-: C6.2, R10.1, USB2.2
- new net VBAT: U5.3
- new net VIN: C24.2, C27.2, CHRG2.4, D4.-, D5.-, LDO2.1, LDO2.3, R14.2
- new net VLIPO: C26.1, CHRG2.3, D4.+, J2.2, R15.2
- new net V_USB: D5.+, U4.15, USB2.1
Other:
- board outline added: 37.9 x 38.1 mm

Commit message: update
Parts:
- removed C10, C11: 300p, LinnesLab-Passives:C0603
- removed C29: 1u, LinnesLab-Passives:C0603
- removed R17: 100k, LinnesLab-Passives:R0603
- removed U5: PCF8523, LinnesLab-Clocks:SO8
- removed XTAL3: 32.7680kHz, LinnesLab-Clocks:2-SMD.NOLEAD.2.0MMTO1.2MM
- added J1: (no value), LinnesLab-Connectors:1X06_1.27MM
- moved R2 76.8 mm to (28.0, 65.1)
- moved R1 76.6 mm to (33.7, 64.7)
- moved C4 46.3 mm to (25.1, 61.3), turned to 90 degrees
- moved R18 45.2 mm to (36.0, 62.0)
- moved R12 42.5 mm to (35.7, 60.1)
- moved LED6 38.5 mm to (39.2, 62.0), turned to 180 degrees
- moved C14 38.2 mm to (64.1, -16.2)
- moved D1 38.2 mm to (61.6, -16.1)
- moved R5 38.2 mm to (59.2, -16.0)
- moved SW4 38.2 mm to (55.5, -16.0)
- moved C6 37.3 mm to (37.7, 57.7), turned to 270 degrees
- moved LED5 36.5 mm to (38.9, 60.2), turned to 180 degrees
- moved U4 36.1 mm to (30.3, 59.1)
- moved C5 33.8 mm to (37.7, 54.5), turned to 270 degrees
- moved JP2 32.3 mm to (26.7, 53.6)
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Connections:
- removed net BATT: R15.1, R16.2
- removed net CD1: SD2.CD1
- removed net CHRG.STAT: CHRG2.1, R14.1
- removed net CS.OLED: U3.13
- removed net DC.OLED: U3.15
- removed net N$21: U5.1, XTAL3.P$2
- removed net RESET.OLED: U3.14
- removed net SD.CS: SD2.2
- removed net SW1: SW1.A1, SW2.A1
- removed net VBAT: U5.3
- new net A4/BATT: R15.1, R16.2, U2.5
- new net A6/TIA: U2.7
- new net A7/PPG: U2.8
- new net D11/SW1: U2.25
- new net D11/SW2: SW1.A1
- new net D15/SW2: SW2.A1, U2.29
- new net D16/CS/OLED: U2.30, U3.13
- new net D27/CHRG.STATUS: CHRG2.1, R14.1, U2.4
- new net D29/LED.CTRL: U2.6
- new net D3/RESETOLED: U2.16, U3.14
- new net D4/DCOLED: U2.17, U3.15
- new net D5/CD1: SD2.CD1, U2.18
- new net D7/SD.CS: SD2.2, U2.20
- net 3.3V: now also R8.2, R9.2; no longer C29.1, R17.2, U5.8
- net GND: no longer C10.2, C11.2, C29.2, R17.1, U5.4
- net N$20: now also U2.15; no longer U5.2, XTAL3.P$1
- net P0.09/NFC1: no longer C11.1
- net P0.10/NFC2: no longer C10.1
- net SCL: now also R8.1; no longer U5.6
- net SDA: now also R9.1; no longer U5.5
Routing:
- net GND: track 0.00 -> 22.6 mm, vias 0 -> 13
- net TXLED: track 0.00 -> 14.3 mm, vias 0 -> 2
- net VLIPO: track 0.00 -> 8.23 mm
- net N$13: track 0.00 -> 8.07 mm
- net RXD.FT: track 0.00 -> 6.41 mm
- net N$2: track 0.00 -> 5.34 mm
- net N$8: track 0.00 -> 4.06 mm
- net 3.3V: track 0.00 -> 3.60 mm
- net N$15: track 0.00 -> 3.57 mm
- net N$5: track 0.00 -> 3.05 mm
- net TXD.FT: track 0.00 -> 2.69 mm
- net N$24: track 0.00 -> 2.32 mm
- net RXLED: track 0.00 -> 1.90 mm
- net USB+: track 0.00 -> 1.75 mm
- net USB-: track 0.00 -> 1.74 mm
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- added copper zone on layer 1, net 3.3V
- added copper zone on layer 16, net GND

Commit message: current
Parts:
- moved C14 72.5 mm to (3.02, 22.7), turned to 180 degrees
- moved D1 71.6 mm to (3.15, 25.3), turned to 0 degrees
- moved R5 70.9 mm to (3.28, 27.7), turned to 0 degrees
- moved SW4 70.5 mm to (3.28, 31.3), turned to 90 degrees
- moved R2 57.6 mm to (5.62, 12.0)
- moved R11 57.4 mm to (11.3, 2.96)
- moved R18 57.4 mm to (12.0, 9.92)
- moved U4 57.4 mm to (6.26, 7.01)
- moved R10 57.4 mm to (11.2, 4.88)
- moved R12 57.4 mm to (11.7, 7.97)
- moved LED6 57.1 mm to (15.5, 10.1)
- moved R1 57.0 mm to (9.76, 13.0)
- moved C4 56.8 mm to (1.82, 9.59), turned to 270 degrees
- moved JP2 56.5 mm to (2.61, 2.55)
- moved LED5 56.5 mm to (15.4, 8.85)
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Routing:
- net USB-: track 1.74 -> 22.7 mm, vias 0 -> 1
- net VIN: track 0.00 -> 19.0 mm
- net TXLED: track 14.3 -> 0.04 mm, vias 2 -> 0
- net VLIPO: track 8.23 -> 22.3 mm
- net USB+: track 1.75 -> 15.1 mm, vias 0 -> 1
- net N$17: track 0.00 -> 8.73 mm
- net N$13: track 8.07 -> 0.01 mm
- net N$6: track 0.00 -> 7.00 mm
- net N$4: track 0.00 -> 6.65 mm
- net N$2: track 5.34 -> 0.00 mm
- net N$15: track 3.57 -> 0.00 mm
- net GND: track 22.6 -> 25.8 mm, vias 13 -> 15
- net N$12: track 1.61 -> 4.15 mm
- net V_USB: track 0.00 -> 2.18 mm
- net 3.3V: track 3.60 -> 5.73 mm, vias 0 -> 1
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
Commit message: update
Parts:
- removed C24, C25: 1u, LinnesLab-Passives:C0603
- removed C26, C27: 4.7u, LinnesLab-Passives:C0603
- removed J1: (no value), LinnesLab-Connectors:1X06_1.27MM
- removed R13: (no value), LinnesLab-Passives:R0603
- removed R14: 100k, LinnesLab-Passives:R0603
- added C11, C20: 1u, LinnesLab-Passives:C0603
- added C21, C22: 4.7u, LinnesLab-Passives:C0603
- added J3: (no value), LinnesLab-Connectors:1X07_1.27MM
- added R21: 5K, LinnesLab-Passives:R0603
- added R22: 100k, LinnesLab-Passives:R0603
- C18: value 2.2uF -> (none); device LinnesLab-Passives:C0402 -> LinnesLab-Passives:C0603
- moved SW4 35.8 mm to (34.8, 14.5)
- moved R5 34.9 mm to (34.0, 11.2), turned to 180 degrees
- moved D1 34.5 mm to (34.0, 9.70), turned to 180 degrees
- moved C14 34.4 mm to (34.2, 8.22), turned to 0 degrees
- moved LDO2 25.0 mm to (11.3, 27.8), flipped to the top, turned to 270 degrees
- moved LED3 21.3 mm to (34.1, 19.3), turned to 270 degrees
- moved LED4 20.9 mm to (35.4, 19.3), turned to 270 degrees
- moved CHRG2 18.5 mm to (2.94, 25.7), flipped to the top, turned to 0 degrees
- moved C9 16.7 mm to (19.1, 23.5), turned to 90 degrees
- moved R3 16.2 mm to (33.9, 22.3), turned to 90 degrees
- moved R4 15.7 mm to (35.2, 22.3), turned to 90 degrees
- moved C8 15.7 mm to (17.8, 23.4), turned to 270 degrees
- moved CORTEX1 14.1 mm to (35.2, 28.4), turned to 270 degrees
- moved SW3 13.5 mm to (35.0, 35.6), turned to 180 degrees
- moved R2 12.9 mm to (18.5, 11.8)
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Connections:
- net !CTS renamed CTS
- removed net !DTR: U4.1
- removed net A4/BATT: R15.1, R16.2, U2.5
- removed net A6/TIA: U2.7
- removed net A7/PPG: U2.8
- removed net D11/SW2: SW1.A1
- removed net D27/CHRG.STATUS: CHRG2.1, R14.1, U2.4
- removed net D29/LED.CTRL: U2.6
- new net 3.3: C12.2, C17.2, C19.2, C4.2, CORTEX1.1, D1.-, LED5.A, LED6.A, R5.2, R8.2, R9.2, SD2.4, U2.11, U3.6, U3.9, U4.14, U4.3
- new net A4/PPG: J3.7, U2.5
- new net A5/TIA: J3.6, U2.6
- new net A7/BATT: R15.1, R16.2, U2.8
- new net CHRG.STAT: CHRG2.1, R22.1, U2.4
- new net D30/LED.CTRL: J3.5, U2.7
- net 3.3V: now also C20.1, J3.4; no longer C12.2, C17.2, C19.2, C25.1, C4.2, CORTEX1.1, D1.-, LED5.A, LED6.A, R5.2, R8.2, R9.2, SD2.4, U2.11, U3.6, U3.9, U4.14, U4.3
- net D11/SW1: now also SW1.A1
- net DTR: now also U4.1
- net GND: now also C11.1, C20.2, C21.2, C22.1, J3.3, R21.1; no longer C24.1, C25.2, C26.2, C27.1, R13.1
- net N$17: now also R21.2; no longer R13.2
- net SCL: now also J3.2
- net SDA: now also J3.1
- net VIN: now also C11.2, C22.2, R22.2; no longer C24.2, C27.2, R14.2
- net VLIPO: now also C21.1; no longer C26.1
Routing:
- net GND: track 25.8 -> 68.3 mm, vias 15 -> 30
- net DTR: track 0.00 -> 36.8 mm, vias 0 -> 2
- net RESET: track 0.00 -> 31.8 mm, vias 0 -> 1
- net SCK: track 0.00 -> 31.2 mm, vias 0 -> 3
- net MOSI: track 0.00 -> 29.0 mm, vias 0 -> 3
- net CHRG.STAT: track 0.00 -> 26.5 mm, vias 0 -> 5
- net D15/SW2: track 0.00 -> 24.7 mm
- net SCL: track 0.00 -> 24.4 mm, vias 0 -> 1
- net VIN: track 19.0 -> 42.3 mm, vias 0 -> 1
- net A7/BATT: track 0.00 -> 23.0 mm, vias 0 -> 2
- net D7/SD.CS: track 0.00 -> 22.7 mm, vias 0 -> 3
- net D11/SW1: track 0.00 -> 21.4 mm
- net SDA: track 0.00 -> 21.0 mm, vias 0 -> 1
- net TXD.NRF: track 0.00 -> 18.6 mm, vias 0 -> 2
- net D16/CS/OLED: track 0.00 -> 17.7 mm, vias 0 -> 2
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- added copper zone on layer 1, net 3.3
- removed copper zone on layer 1, net 3.3V
Other:
- board text added: "+"

Commit message: check
Routing:
- net D5/CD1: track 0.00 -> 13.8 mm, vias 0 -> 1
- net MOSI: track 29.0 -> 32.3 mm
- net SCK: track 31.2 -> 33.9 mm
- net TXD.NRF: track 18.6 -> 20.0 mm
- net D4/DCOLED: track 12.2 -> 13.2 mm
- net D3/RESETOLED: track 11.8 -> 12.9 mm
- net N$4: track 7.84 -> 6.90 mm
- net TXLED: track 11.2 -> 10.6 mm

Commit message: saved
Parts:
- moved R6 1.71 mm to (16.4, 24.1)
- moved C7 0.87 mm to (16.9, 30.3)
- moved C12 0.45 mm to (17.5, 32.2)
- moved L2 0.45 mm to (17.5, 28.9)
- moved R15 0.33 mm to (4.18, 20.1)
Routing:
- net 3.3: track 9.24 -> 73.1 mm, vias 1 -> 5
- net GND: track 68.4 -> 78.4 mm, vias 30 -> 31
- net CHRG.STAT: track 26.5 -> 30.2 mm
- net D15/SW2: track 24.7 -> 27.3 mm, vias 0 -> 2
- net N$1: track 2.19 -> 3.92 mm
- net D4/DCOLED: track 13.2 -> 15.0 mm
- net D3/RESETOLED: track 12.9 -> 14.1 mm
- net D16/CS/OLED: track 17.7 -> 18.8 mm
- net SCK: track 33.9 -> 34.7 mm
- net N$12: track 6.64 -> 7.20 mm
- net D11/SW1: track 21.3 -> 20.7 mm
- added copper zone on layer 1, net 3.3V
- removed copper zone on layer 1, net 3.3
